Commit message: feat: add gazebo simulation

File: ros2/kachaka_description/robot/kachaka.urdf.xacro (robot description, xacro)
@@ -1,7 +1,7 @@
 <?xml version="1.0"?>
-<robot name="kachaka"
-       xmlns:xacro="http://ros.org/wiki/xacro">
+<robot name="kachaka" xmlns:xacro="http://ros.org/wiki/xacro">
   <xacro:include filename="$(find kachaka_description)/urdf/_materials.urdf.xacro" />
   <xacro:include filename="$(find kachaka_description)/urdf/_values.urdf.xacro" />
+  <xacro:include filename="$(find kachaka_description)/urdf/_kachaka.gazebo.xacro" />
   <xacro:include filename="$(find kachaka_description)/urdf/_kachaka.urdf.xacro" />
   <link name="base_footprint" />

File: ros2/kachaka_description/urdf/_kachaka.urdf.xacro (robot description, xacro)
@@ -127,5 +127,5 @@
       <parent link="base_link" />
       <child link="camera_front_link" />
-      <origin rpy="-${PI / 2.0} 0 -${PI / 2.0}"
+      <origin rpy="0 0 0"
               xyz="${0.2196 - 0.01} 0 0.070" />
     </joint>
@@ -136,5 +136,5 @@
       <parent link="base_link" />
       <child link="camera_back_link" />
-      <origin rpy="-${PI / 2.0} 0 ${PI / 2.0}"
+      <origin rpy="0 0 ${PI}"
               xyz="${-0.150 + 0.01} 0 0.070" />
     </joint>
@@ -145,5 +145,5 @@
       <parent link="base_link" />
       <child link="tof_link" />
-      <origin rpy="-${PI / 4.0} 0 -${PI / 2.0}"
+      <origin rpy=" 0 -${PI / 4.0} 0"
               xyz="0.221 0.0 0.0418" />
     </joint>
